Commit message: prime

File: urdf/robot.xacro (robot description, xacro)
@@ -1,384 +1,384 @@
 <?xml version="1.0" ?>
 <robot name="robot">
-    <link name="link_base">
-    <inertial>
-      <origin xyz="0 0 0" rpy="0 0 0"/>
-      <mass value="0.1"/>
-      <inertia ixx="0.001" ixy="0" ixz="0" iyy="0.001" iyz="0" izz="0.001"/>
-    </inertial>
-        <visual>
-      <origin xyz="0 0 0" rpy="0 0 0"/>
-      <geometry>
-        <mesh filename="$(find robot)/mesh/assets/part_8.stl" scale="0.1 0.1 0.1"/>
-      </geometry>
-      <material name="part_8_material">
-        <color rgba="0.231373 0.380392 0.705882 1.0"/>
-      </material>
-    </visual>
-    <collision>
-      <origin xyz="0 0 0" rpy="0 0 0"/>
-      <geometry>
-        <mesh filename="$(find robot)/mesh/assets/part_8.stl" scale="0.1 0.1 0.1"/>
-      </geometry>
-    </collision>
-        <visual>
-      <origin xyz="0 0 0" rpy="0 0 0"/>
-      <geometry>
-        <mesh filename="$(find robot)/mesh/assets/part_14.stl" scale="0.1 0.1 0.1"/>
-      </geometry>
-      <material name="part_14_material">
-        <color rgba="0.615686 0.811765 0.929412 1.0"/>
-      </material>
-    </visual>
-    <collision>
-      <origin xyz="0 0 0" rpy="0 0 0"/>
-      <geometry>
-        <mesh filename="$(find robot)/mesh/assets/part_14.stl" scale="0.1 0.1 0.1"/>
-      </geometry>
-    </collision>
-        <visual>
-      <origin xyz="0 0 0" rpy="0 0 0"/>
-      <geometry>
-        <mesh filename="$(find robot)/mesh/assets/part_20.stl" scale="0.1 0.1 0.1"/>
-      </geometry>
-      <material name="part_20_material">
-        <color rgba="0.498039 0.498039 0.498039 1.0"/>
-      </material>
-    </visual>
-    <collision>
-      <origin xyz="0 0 0" rpy="0 0 0"/>
-      <geometry>
-        <mesh filename="$(find robot)/mesh/assets/part_20.stl" scale="0.1 0.1 0.1"/>
-      </geometry>
-    </collision>
-        <visual>
-      <origin xyz="0 0 0" rpy="0 0 0"/>
-      <geometry>
-        <mesh filename="$(find robot)/mesh/assets/part_6.stl" scale="0.1 0.1 0.1"/>
-      </geometry>
-      <material name="part_6_material">
-        <color rgba="0.615686 0.811765 0.929412 1.0"/>
-      </material>
-    </visual>
-    <collision>
-      <origin xyz="0 0 0" rpy="0 0 0"/>
-      <geometry>
-        <mesh filename="$(find robot)/mesh/assets/part_6.stl" scale="0.1 0.1 0.1"/>
-      </geometry>
-    </collision>
-        <visual>
-      <origin xyz="0 0 0" rpy="0 0 0"/>
-      <geometry>
-        <mesh filename="$(find robot)/mesh/assets/part_18.stl" scale="0.1 0.1 0.1"/>
-      </geometry>
-      <material name="part_18_material">
-        <color rgba="0.768627 0.886275 0.952941 1.0"/>
-      </material>
-    </visual>
-    <collision>
-      <origin xyz="0 0 0" rpy="0 0 0"/>
-      <geometry>
-        <mesh filename="$(find robot)/mesh/assets/part_18.stl" scale="0.1 0.1 0.1"/>
-      </geometry>
-    </collision>
-        <visual>
-      <origin xyz="0 0 0" rpy="0 0 0"/>
-      <geometry>
-        <mesh filename="$(find robot)/mesh/assets/part_9.stl" scale="0.1 0.1 0.1"/>
-      </geometry>
-      <material name="part_9_material">
-        <color rgba="0.917647 0.917647 0.917647 1.0"/>
-      </material>
-    </visual>
-    <collision>
-      <origin xyz="0 0 0" rpy="0 0 0"/>
-      <geometry>
-        <mesh filename="$(find robot)/mesh/assets/part_9.stl" scale="0.1 0.1 0.1"/>
-      </geometry>
-    </collision>
-        <visual>
-      <origin xyz="0 0 0" rpy="0 0 0"/>
-      <geometry>
-        <mesh filename="$(find robot)/mesh/assets/part_16.stl" scale="0.1 0.1 0.1"/>
-      </geometry>
-      <material name="part_16_material">
-        <color rgba="0.231373 0.380392 0.705882 1.0"/>
-      </material>
-    </visual>
-    <collision>
-      <origin xyz="0 0 0" rpy="0 0 0"/>
-      <geometry>
-        <mesh filename="$(find robot)/mesh/assets/part_16.stl" scale="0.1 0.1 0.1"/>
-      </geometry>
-    </collision>
-        <visual>
-      <origin xyz="0 0 0" rpy="0 0 0"/>
-      <geometry>
-        <mesh filename="$(find robot)/mesh/assets/part_5.stl" scale="0.1 0.1 0.1"/>
-      </geometry>
-      <material name="part_5_material">
-        <color rgba="0.980392 0.713725 0.00392157 1.0"/>
-      </material>
-    </visual>
-    <collision>
-      <origin xyz="0 0 0" rpy="0 0 0"/>
-      <geometry>
-        <mesh filename="$(find robot)/mesh/assets/part_5.stl" scale="0.1 0.1 0.1"/>
-      </geometry>
-    </collision>
-        <visual>
-      <origin xyz="0 0 0" rpy="0 0 0"/>
-      <geometry>
-        <mesh filename="$(find robot)/mesh/assets/part_2.stl" scale="0.1 0.1 0.1"/>
-      </geometry>
-      <material name="part_2_material">
-        <color rgba="0.768627 0.886275 0.952941 1.0"/>
-      </material>
-    </visual>
-    <collision>
-      <origin xyz="0 0 0" rpy="0 0 0"/>
-      <geometry>
-        <mesh filename="$(find robot)/mesh/assets/part_2.stl" scale="0.1 0.1 0.1"/>
-      </geometry>
-    </collision>
-        <visual>
-      <origin xyz="0 0 0" rpy="0 0 0"/>
-      <geometry>
-        <mesh filename="$(find robot)/mesh/assets/part_4.stl" scale="0.1 0.1 0.1"/>
-      </geometry>
-      <material name="part_4_material">
-        <color rgba="0.498039 0.498039 0.498039 1.0"/>
-      </material>
-    </visual>
-    <collision>
-      <origin xyz="0 0 0" rpy="0 0 0"/>
-      <geometry>
-        <mesh filename="$(find robot)/mesh/assets/part_4.stl"  scale="0.1 0.1 0.1"/>
-      </geometry>
-    </collision>
-        <visual>
-      <origin xyz="0 0 0" rpy="0 0 0"/>
-      <geometry>
-        <mesh filename="$(find robot)/mesh/assets/part_11.stl" scale="0.1 0.1 0.1"/>
-      </geometry>
-      <material name="part_11_material">
-        <color rgba="0.972549 0.529412 0.00392157 1.0"/>
-      </material>
-    </visual>
-    <collision>
-      <origin xyz="0 0 0" rpy="0 0 0"/>
-      <geometry>
-        <mesh filename="$(find robot)/mesh/assets/part_11.stl" scale="0.1 0.1 0.1"/>
-      </geometry>
-    </collision>
-        <visual>
-      <origin xyz="0 0 0" rpy="0 0 0"/>
-      <geometry>
-        <mesh filename="$(find robot)/mesh/assets/part_10.stl" scale="0.1 0.1 0.1"/>
-      </geometry>
-      <material name="part_10_material">
-        <color rgba="0.768627 0.886275 0.952941 1.0"/>
-      </material>
-    </visual>
-    <collision>
-      <origin xyz="0 0 0" rpy="0 0 0"/>
-      <geometry>
-        <mesh filename="$(find robot)/mesh/assets/part_10.stl" scale="0.1 0.1 0.1"/>
-      </geometry>
-    </collision>
-        <visual>
-      <origin xyz="0 0 0" rpy="0 0 0"/>
-      <geometry>
-        <mesh filename="$(find robot)/mesh/assets/part_15.stl" scale="0.1 0.1 0.1"/>
-      </geometry>
-      <material name="part_15_material">
-        <color rgba="0.647059 0.647059 0.647059 1.0"/>
-      </material>
-    </visual>
-    <collision>
-      <origin xyz="0 0 0" rpy="0 0 0"/>
-      <geometry>
-        <mesh filename="$(find robot)/mesh/assets/part_15.stl" scale="0.1 0.1 0.1"/>
-      </geometry>
-    </collision>
-        <visual>
-      <origin xyz="0 0 0" rpy="0 0 0"/>
-      <geometry>
-        <mesh filename="$(find robot)/mesh/assets/part_3.stl" scale="0.1 0.1 0.1"/>
-      </geometry>
-      <material name="part_3_material">
-        <color rgba="0.972549 0.529412 0.00392157 1.0"/>
-      </material>
-    </visual>
-    <collision>
-      <origin xyz="0 0 0" rpy="0 0 0"/>
-      <geometry>
-        <mesh filename="$(find robot)/mesh/assets/part_3.stl" scale="0.1 0.1 0.1"/>
-      </geometry>
-    </collision>
-        <visual>
-      <origin xyz="0 0 0" rpy="0 0 0"/>
-      <geometry>
-        <mesh filename="$(find robot)/mesh/assets/part_7.stl" scale="0.1 0.1 0.1"/>
-      </geometry>
-      <material name="part_7_material">
-        <color rgba="0.647059 0.647059 0.647059 1.0"/>
-      </material>
-    </visual>
-    <collision>
-      <origin xyz="0 0 0" rpy="0 0 0"/>
-      <geometry>
-        <mesh filename="$(find robot)/mesh/assets/part_7.stl" scale="0.1 0.1 0.1"/>
-      </geometry>
-    </collision>
-        <visual>
-      <origin xyz="0 0 0" rpy="0 0 0"/>
-      <geometry>
-        <mesh filename="$(find robot)/mesh/assets/part_17.stl" scale="0.1 0.1 0.1"/>
-      </geometry>
-      <material name="part_17_material">
-        <color rgba="0.917647 0.917647 0.917647 1.0"/>
-      </material>
-    </visual>
-    <collision>
-      <origin xyz="0 0 0" rpy="0 0 0"/>
-      <geometry>
-        <mesh filename="$(find robot)/mesh/assets/part_17.stl" scale="0.1 0.1 0.1"/>
-      </geometry>
-    </collision>
-        <visual>
-      <origin xyz="0 0 0" rpy="0 0 0"/>
-      <geometry>
-        <mesh filename="$(find robot)/mesh/assets/part_1.stl" scale="0.1 0.1 0.1"/>
-      </geometry>
-      <material name="part_1_material">
-        <color rgba="0.917647 0.917647 0.917647 1.0"/>
-      </material>
-    </visual>
-    <collision>
-      <origin xyz="0 0 0" rpy="0 0 0"/>
-      <geometry>
-        <mesh filename="$(find robot)/mesh/assets/part_1.stl" scale="0.1 0.1 0.1"/>
-      </geometry>
-    </collision>
-        <visual>
-      <origin xyz="0 0 0" rpy="0 0 0"/>
-      <geometry>
-        <mesh filename="$(find robot)/mesh/assets/part_13.stl" scale="0.1 0.1 0.1"/>
-      </geometry>
-      <material name="part_13_material">
-        <color rgba="0.980392 0.713725 0.00392157 1.0"/>
-      </material>
-    </visual>
-    <collision>
-      <origin xyz="0 0 0" rpy="0 0 0"/>
-      <geometry>
-        <mesh filename="$(find robot)/mesh/assets/part_13.stl" scale="0.1 0.1 0.1"/>
-      </geometry>
-    </collision>
-        <visual>
-      <origin xyz="0 0 0" rpy="0 0 0"/>
-      <geometry>
-        <mesh filename="$(find robot)/mesh/assets/part_19.stl" scale="0.1 0.1 0.1"/>
-      </geometry>
-      <material name="part_19_material">
-        <color rgba="0.972549 0.529412 0.00392157 1.0"/>
-      </material>
-    </visual>
-    <collision>
-      <origin xyz="0 0 0" rpy="0 0 0"/>
-      <geometry>
-        <mesh filename="$(find robot)/mesh/assets/part_19.stl" scale="0.1 0.1 0.1"/>
-      </geometry>
-    </collision>
-        <visual>
-      <origin xyz="0 0 0" rpy="0 0 0"/>
-      <geometry>
-        <mesh filename="$(find robot)/mesh/assets/part_12.stl" scale="0.1 0.1 0.1"/>
-      </geometry>
-      <material name="part_12_material">
-        <color rgba="0.498039 0.498039 0.498039 1.0"/>
-      </material>
-    </visual>
-    <collision>
-      <origin xyz="0 0 0" rpy="0 0 0"/>
-      <geometry>
-        <mesh filename="$(find robot)/mesh/assets/part_12.stl" scale="0.1 0.1 0.1"/>
-      </geometry>
-    </collision>
-  </link>
-    <link name="link_hip_l">
-    <inertial>
-      <origin xyz="0 0 0" rpy="0 0 0"/>
-      <mass value="0.1"/>
-      <inertia ixx="0.001" ixy="0" ixz="0" iyy="0.001" iyz="0" izz="0.001"/>
-    </inertial>
-        <visual>
-      <origin xyz="0 0 0" rpy="0 0 0"/>
-      <geometry>
-        <mesh filename="$(find robot)/mesh/assets/part_2__2.stl" scale="0.1 0.1 0.1"/>
-      </geometry>
-      <material name="part_2_2_material">
-        <color rgba="0.231373 0.380392 0.705882 1.0"/>
-      </material>
-    </visual>
-    <collision>
-      <origin xyz="0 0 0" rpy="0 0 0"/>
-      <geometry>
-        <mesh filename="$(find robot)/mesh/assets/part_2__2.stl" scale="0.1 0.1 0.1"/>
-      </geometry>
-    </collision>
-        <visual>
-      <origin xyz="0 0 0" rpy="0 0 0"/>
-      <geometry>
-        <mesh filename="$(find robot)/mesh/assets/part_3__2.stl" scale="0.1 0.1 0.1"/>
-      </geometry>
-      <material name="part_3_2_material">
-        <color rgba="0.917647 0.917647 0.917647 1.0"/>
-      </material>
-    </visual>
-    <collision>
-      <origin xyz="0 0 0" rpy="0 0 0"/>
-      <geometry>
-        <mesh filename="$(find robot)/mesh/assets/part_3__2.stl" scale="0.1 0.1 0.1"/>
-      </geometry>
-    </collision>
-        <visual>
-      <origin xyz="0 0 0" rpy="0 0 0"/>
-      <geometry>
-        <mesh filename="$(find robot)/mesh/assets/part_4__2.stl" scale="0.1 0.1 0.1"/>
-      </geometry>
-      <material name="part_4_2_material">
-        <color rgba="0.768627 0.886275 0.952941 1.0"/>
-      </material>
-    </visual>
-    <collision>
-      <origin xyz="0 0 0" rpy="0 0 0"/>
-      <geometry>
-        <mesh filename="$(find robot)/mesh/assets/part_4__2.stl" scale="0.1 0.1 0.1"/>
-      </geometry>
-    </collision>
-        <visual>
-      <origin xyz="0 0 0" rpy="0 0 0"/>
-      <geometry>
-        <mesh filename="$(find robot)/mesh/assets/part_1__2.stl" scale="0.1 0.1 0.1"/>
-      </geometry>
-      <material name="part_1_2_material">
-        <color rgba="0.647059 0.647059 0.647059 1.0"/>
-      </material>
-    </visual>
-    <collision>
-      <origin xyz="0 0 0" rpy="0 0 0"/>
-      <geometry>
-        <mesh filename="$(find robot)/mesh/assets/part_1__2.stl" scale="0.1 0.1 0.1"/>
-      </geometry>
-    </collision>
-  </link>
-    <joint name="joint12" type="fixed">
-    <origin xyz="0 0 0" rpy="0 0 0"/>
-    <parent link="link_base"/>
-    <child link="link_hip_l"/>
-    <axis xyz="0 0 1"/>
-    <limit effort="10" velocity="10"/>
-  </joint>
+    <link name="link_base">
+    <inertial>
+      <origin xyz="0 0 0" rpy="0 0 0"/>
+      <mass value="0.1"/>
+      <inertia ixx="0.001" ixy="0" ixz="0" iyy="0.001" iyz="0" izz="0.001"/>
+    </inertial>
+        <visual>
+      <origin xyz="0 0 0" rpy="0 0 0"/>
+      <geometry>
+        <mesh filename="$(find robot)/meshes/assets/part_8.stl"/>
+      </geometry>
+      <material name="part_8_material">
+        <color rgba="0.231373 0.380392 0.705882 1.0"/>
+      </material>
+    </visual>
+    <collision>
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